File: Electronics/TechBird-SmartSense/TechBird_SmartTemp.kicad_pcb (KiCad board)
At the start: 2 copper layers, 50 x 40 mm, 80 parts, among them J1 UJ20-C-H-G-SMT-P16-TR, J2 S2B-PH-SM4, J3 1771088, SW1 SKRPARE010, SW2 SKRPARE010, U1 USBLC6-2SC6, U2 TMP1075D, U3 BQ21040DBVR, U4 TLV75733PDBV, U5 REF3033, U6 ESP32-C6-MINI-1-N4, U7 RV-3028-C7, U8 FM24C64B-G, U9 ADS1015IDGSR

Commit message: Initial Push for 003
Parts:
- removed C15: 100m, Capacitor_THT:CP_Radial_Tantal_D10.5mm_P5.00mm
- removed TP10, TP4, TP6, TP7, TP8, TP9: TestPoint, TestPoint:TestPoint_Pad_D1.0mm
- added C16: 10u, Capacitor_SMD:C_0603_1608Metric, F.Cu at (144.5, 81.0)
- added C17: 100n, Capacitor_SMD:C_0603_1608Metric, F.Cu at (140.3, 81.0)
- added C19: 100n, Resistor_SMD:R_0603_1608Metric, F.Cu at (91.0, 79.9)
- added C20: 10u, Capacitor_SMD:C_0603_1608Metric, F.Cu at (98.0, 75.9)
- added C21: 10u, Resistor_SMD:R_0805_2012Metric, F.Cu at (91.0, 81.7)
- added C22: 10u, Resistor_SMD:R_0805_2012Metric, F.Cu at (91.0, 83.7)
- added C23: 10u, Resistor_SMD:R_0805_2012Metric, F.Cu at (91.0, 85.7)
- added C24: 100n, Resistor_SMD:R_0603_1608Metric, F.Cu at (94.5, 85.9)
- added C25: 10u, Capacitor_SMD:C_0603_1608Metric, F.Cu at (99.6, 75.9)
- added C26: 10u, Capacitor_SMD:C_0603_1608Metric, F.Cu at (101.2, 75.9)
- added C27: 10u, Capacitor_SMD:C_0603_1608Metric, F.Cu at (90.3, 75.9)
- added C28: 10u, Capacitor_SMD:C_0603_1608Metric, F.Cu at (91.9, 75.9)
- added C29: 10u, Capacitor_SMD:C_0603_1608Metric, F.Cu at (93.5, 75.9)
- added C30: 100n, Capacitor_SMD:C_0603_1608Metric, F.Cu at (102.8, 75.9)
- added C31: 100n, Capacitor_SMD:C_0603_1608Metric, F.Cu at (95.1, 75.9)
- added D4: F.0603.00139/P2-0603R1TS2-06T-002, LED_SMD:LED_0603_1608Metric, F.Cu at (113.6, 61.7)
- added D6: LTST-C193TBKT-5A, LED_SMD:LED_0603_1608Metric, F.Cu at (98.6, 58.9)
- added F1: BSMD1812-200-30V, Fuse:Fuse_1812_4532Metric, F.Cu at (92.3, 88.8)
- added J4: S2B-PH-SM4, Connector_JST:JST_PH_S2B-PH-SM4-TB_1x02-1MP_P2.00mm_Horizontal, F.Cu at (119.0, 92.2)
- added J5: S2B-PH-SM4, Connector_JST:JST_PH_S2B-PH-SM4-TB_1x02-1MP_P2.00mm_Horizontal, F.Cu at (128.5, 92.2)
- added J6: S2B-PH-SM4, Connector_JST:JST_PH_S2B-PH-SM4-TB_1x02-1MP_P2.00mm_Horizontal, F.Cu at (138.0, 92.2)
- added J7: TF-01A, TB_Connectors:HRO TF-01A, F.Cu at (144.1, 72.0)
- added J8: S2B-PH-SM4, Connector_JST:JST_PH_S2B-PH-SM4-TB_1x02-1MP_P2.00mm_Horizontal, F.Cu at (100.0, 92.2)
- added JP2: SolderJumper_2_Open, Jumper:SolderJumper-2_P1.3mm_Open_TrianglePad1.0x1.5mm, F.Cu at (105.6, 86.4)
- added JP3: SolderJumper_2_Open, Jumper:SolderJumper-2_P1.3mm_Open_TrianglePad1.0x1.5mm, F.Cu at (97.8, 61.8)
- added L1: 6.8u, Inductor_SMD:L_Chilisin_BMRx00060630, F.Cu at (100.0, 82.5)
- added R32: 22, Resistor_SMD:R_0603_1608Metric, F.Cu at (119.8, 69.8)
- added R33: 22, Resistor_SMD:R_0603_1608Metric, F.Cu at (121.5, 69.8)
- added R34: 10k, Resistor_SMD:R_0603_1608Metric, F.Cu at (133.8, 69.6)
- added R35: 10k, Resistor_SMD:R_0603_1608Metric, F.Cu at (133.8, 71.2)
- added R36: 10k, Resistor_SMD:R_0603_1608Metric, F.Cu at (133.8, 73.0)
- added R37: 10k, Resistor_SMD:R_0603_1608Metric, F.Cu at (133.8, 74.6)
- added R38: 10k, Resistor_SMD:R_0603_1608Metric, F.Cu at (133.8, 76.3)
- added R39: 22, Resistor_SMD:R_0603_1608Metric, F.Cu at (130.7, 69.6)
- added R40: 22, Resistor_SMD:R_0603_1608Metric, F.Cu at (130.7, 71.2)
- added R41: 22, Resistor_SMD:R_0603_1608Metric, F.Cu at (130.7, 73.0)
- added R42: 22, Resistor_SMD:R_0603_1608Metric, F.Cu at (130.7, 74.6)
- added R43: 22, Resistor_SMD:R_0603_1608Metric, F.Cu at (130.7, 76.3)
- added R44: 22, Resistor_SMD:R_0603_1608Metric, F.Cu at (130.7, 77.9)
- added R45: 10k, Resistor_SMD:R_0603_1608Metric, F.Cu at (133.8, 77.9)
- added R46: 10k, Resistor_SMD:R_0603_1608Metric, F.Cu at (133.8, 79.6)
- added R47: 47k, Resistor_SMD:R_0603_1608Metric, F.Cu at (94.5, 78.3)
- added R48: 10k, Resistor_SMD:R_0603_1608Metric, F.Cu at (91.0, 78.3)
- added R51: 53.6k, Resistor_SMD:R_0603_1608Metric, F.Cu at (94.5, 79.9)
- added R52: 10.2k, Resistor_SMD:R_0603_1608Metric, F.Cu at (94.5, 81.5)
- added R54: 560, Resistor_SMD:R_0603_1608Metric, F.Cu at (97.0, 58.9)
- added U10: TPS563300, Package_TO_SOT_SMD:SOT-583-8, F.Cu at (94.5, 83.7)
- C18: value 1u -> 100n
- J2: footprint 000_Connector:JST_S2B-PH-SM4-TB -> Connector_JST:JST_PH_S2B-PH-SM4-TB_1x02-1MP_P2.00mm_Horizontal
- J3: value 1771088 -> S2B-PH-SM4; footprint TB_Connectors:PHOENIX_1771088 -> Connector_JST:JST_PH_S2B-PH-SM4-TB_1x02-1MP_P2.00mm_Horizontal
- R27: value 0 -> 280
- U8: value FM24C64B-G -> FM24CL64B-GTR
- moved C10 53.0 mm to (145.1, 85.6), turned to -90 degrees
- moved U5 50.3 mm to (142.5, 86.1), turned to -90 degrees
- moved C11 48.3 mm to (139.9, 85.6), turned to -90 degrees
- moved R18 46.4 mm to (137.9, 83.8), turned to 90 degrees
- moved J1 45.7 mm to (91.2, 68.4), turned to -90 degrees
- moved R17 45.1 mm to (136.3, 83.8), turned to 90 degrees
- moved C14 44.0 mm to (134.7, 83.8), turned to 90 degrees
- moved U9 37.6 mm to (132.0, 83.9), turned to -90 degrees
- moved C1 34.2 mm to (97.8, 63.9), turned to 0 degrees
- moved R26 33.2 mm to (97.8, 71.3), turned to 0 degrees
- moved R27 33.1 mm to (113.6, 64.8), turned to 90 degrees
- moved U1 31.7 mm to (98.3, 68.4), turned to 180 degrees
- moved R25 30.9 mm to (97.8, 65.5), turned to 0 degrees
- moved R5 29.3 mm to (128.6, 81.5), turned to 180 degrees
- moved R28 24.7 mm to (125.5, 81.5), turned to 0 degrees
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Connections:
- net /X_USB_D+ renamed /USB/X_USB_D+
- net /X_USB_D- renamed /USB/X_USB_D-
- J3 pad 1: ADC_CH1 -> /I2C Devices/AIN1
- R10 pad 1: /HEARTBEAT -> Net-(U6-IO1)
- R13 pad 2: ~{ALERT} -> Net-(U2-ALERT)
- R20 pad 1: +3.3V -> Net-(JP2-A)
- R21 pad 2: USB_DETECT -> /USB/USB.DETECT
- R22 pad 1: USB_DETECT -> /USB/USB.DETECT
- R23 pad 2: ADC_CH3 -> /I2C Devices/AIN2
- R24 pad 2: ADC_CH4 -> /I2C Devices/AIN3
- R27 pad 1: Net-(U7-VBACKUP) -> Net-(U6-IO0)
- R28 pad 2: ADC_CH1 -> /I2C Devices/AIN0
- R29 pad 2: ADC_CH2 -> /I2C Devices/AIN1
- R30 pad 2: ADC_CH3 -> /I2C Devices/AIN2
- R31 pad 2: ADC_CH4 -> /I2C Devices/AIN3
- R5 pad 2: ADC_CH1 -> /I2C Devices/AIN0
- R7 pad 2: ADC_CH2 -> /I2C Devices/AIN1
- TP5 pad 1: Net-(U6-IO1) -> Net-(U7-VBACKUP)
- U2 pad 3: ~{ALERT} -> Net-(U2-ALERT)
- U6 pad 10: Net-(U6-IO5) -> +3.3VA
- U6 pad 17: USB_D- -> Net-(U6-IO12)
- U6 pad 18: USB_D+ -> Net-(U6-IO13)
- U6 pad 19: Net-(U6-IO14) -> ~{CHARGE}
- U6 pad 20: Net-(U6-IO15) -> CLKOUT
- U6 pad 24: ~{CHARGE} -> SDIO.CMD
- U6 pad 25: USB_DETECT -> SDIO.CLK
- U6 pad 26: CLKOUT -> SDIO.DATA0
- U6 pad 27: ~{ALERT} -> SDIO.DATA1
- U6 pad 28: ~{WKUP} -> SDIO.DATA2
- U6 pad 29: /HEARTBEAT -> SDIO.DATA3
- U6 pad 5: Net-(U6-IO2) -> ~{WKUP}
- U6 pad 9: Net-(U6-IO4) -> SD.DETECT
- U9 pad 4: ADC_CH1 -> /I2C Devices/AIN0
- U9 pad 5: ADC_CH2 -> /I2C Devices/AIN1
- U9 pad 6: ADC_CH3 -> /I2C Devices/AIN2
- U9 pad 7: ADC_CH4 -> /I2C Devices/AIN3
Routing:
- net LP_I2C_SCL: track 59.9 -> 0.00 mm, vias 5 -> 0
- net LP_I2C_SDA: track 58.7 -> 0.00 mm, vias 5 -> 0
- net +3.3V: track 123.5 -> 78.0 mm, vias 7 -> 6
- net +5V: track 26.4 -> 65.9 mm
- net +BATT: track 56.3 -> 18.1 mm
- net ADC_CH4: track 30.0 -> 0.00 mm
- net ~{WKUP}: track 31.1 -> 2.17 mm, vias 2 -> 0
- net +3.3VA: track 44.8 -> 16.0 mm, vias 5 -> 0
- net ~{ALERT}: track 26.2 -> 0.00 mm, vias 2 -> 0
- net CLKOUT: track 25.5 -> 0.00 mm, vias 2 -> 0
- net ADC_CH3: track 23.0 -> 0.00 mm
- net ~{CHARGE}: track 22.6 -> 4.26 mm, vias 2 -> 0
- net ADC_CH2: track 14.6 -> 0.00 mm
- net Net-(U10-VIN): track 0.00 -> 14.1 mm
- net Net-(U10-EN): track 0.00 -> 11.9 mm
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Other:
- board size 50 x 40 mm -> 60 x 40 mm
