File: Electronics/TechBird-SmartSense/TechBird_SmartTemp.kicad_sch (KiCad schematic)
At the start: 80 parts, among them J1 UJ20-C-H-G-SMT-P16-TR, J2 S2B-PH-SM4, J3 1771088, SW1 SKRPARE010, SW2 SKRPARE010, U1 USBLC6-2SC6, U2 TMP1075D, U3 BQ21040DBVR, U4 TLV75733PDBV, U5 REF3033, U6 ESP32-C6-MINI-1-N4, U7 RV-3028-C7, U8 FM24CL64B-GTR, U9 ADS1015IDGSR

Commit message: Initial Push for 003
Parts:
- removed C1, C10, C11, C12, C13, C14, C2, C3, C5, C7: 100n, Capacitor_SMD:C_0603_1608Metric, symbol Device:C
- removed C15: 100m, Capacitor_THT:CP_Radial_Tantal_D10.5mm_P5.00mm, symbol Device:C_Polarized
- removed C4: 1u, Capacitor_SMD:C_0603_1608Metric, symbol Device:C
- removed C6: 10u, Capacitor_SMD:C_0603_1608Metric, symbol Device:C
- removed D1, D3: LTST-C193TBKT-5A, LED_SMD:LED_0603_1608Metric, symbol Device:LED
- removed J1: UJ20-C-H-G-SMT-P16-TR, Connector_USB:USB_C_Receptacle_G-Switch_GT-USB-7010ASV, symbol Connector:USB_C_Receptacle_USB2.0_16P
- removed J2: S2B-PH-SM4, 000_Connector:JST_S2B-PH-SM4-TB, symbol Connector_Generic:Conn_01x02
- removed J3: 1771088, TB_Connectors:PHOENIX_1771088, symbol Connector_Generic:Conn_01x08
- removed R1: 280, Resistor_SMD:R_0603_1608Metric, symbol Device:R
- removed R11, R13, R14, R15, R16, R17, R18, R2, R21: 10k, Resistor_SMD:R_0603_1608Metric, symbol Device:R
- removed R20: 100, Resistor_SMD:R_0603_1608Metric, symbol Device:R
- removed R22: 6.8k, Resistor_SMD:R_0603_1608Metric, symbol Device:R
- removed R23, R24, R3, R5, R7: 1.5k, Resistor_SMD:R_0603_1608Metric, symbol Device:R
- removed R25, R26: 5.1k, Resistor_SMD:R_0603_1608Metric, symbol Device:R
- removed R28, R29, R30, R31: 0, Resistor_SMD:R_0603_1608Metric, symbol Device:R
- removed R4: 24k, Resistor_SMD:R_0603_1608Metric, symbol Device:R
- removed TP10, TP3, TP4, TP5, TP6, TP7, TP8, TP9: TestPoint, TestPoint:TestPoint_Pad_D1.0mm, symbol Connector:TestPoint
- removed U1: USBLC6-2SC6, Package_TO_SOT_SMD:SOT-23-6, symbol Power_Protection:USBLC6-2SC6
- removed U2: TMP1075D, Package_SO:SOIC-8_3.9x4.9mm_P1.27mm, symbol Sensor_Temperature:TMP1075D
- removed U3: BQ21040DBVR, Package_TO_SOT_SMD:SOT-23-6, symbol 000_Power:BQ21040DBVR
- removed U4: TLV75733PDBV, Package_TO_SOT_SMD:SOT-23-5, symbol Regulator_Linear:TLV75733PDBV
- removed U5: REF3033, Package_TO_SOT_SMD:SOT-23, symbol Reference_Voltage:REF3033
- removed U7: RV-3028-C7, Package_SON:MicroCrystal_C7_SON-8_1.5x3.2mm_P0.9mm, symbol Timer_RTC:RV-3028-C7
- removed U8: FM24CL64B-GTR, Package_SO:SOIC-8_3.9x4.9mm_P1.27mm, symbol Memory_NVRAM:FM24C64B
- removed U9: ADS1015IDGSR, Package_SO:TSSOP-10_3x3mm_P0.5mm, symbol Analog_ADC:ADS1015IDGS
- added D4: F.0603.00139/P2-0603R1TS2-06T-002, LED_SMD:LED_0603_1608Metric, symbol Device:LED
- added R32, R33: 22, Resistor_SMD:R_0603_1608Metric, symbol Device:R
- C18: value 1u -> 100n; DigiKey 445-C1608X7R1C105K080DCCT-ND -> 399-C0603C104K3RACTUCT-ND; Distri Link https://www.digikey.de/de/products/detail/tdk-corporation/C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 -> https://www.digikey.de/de/products/detail/kemet/C0603C104K3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; MFG TDK Corporation -> KEMET; MFG# C1608X7R1C105K080DC -> C0603C104K3RACTU
- R27: value 0 -> 280; DigiKey CR0603AJ/-000EASCT-ND -> 311-280HRCT-ND; Distri Link https://www.digikey.de/de/products/detail/bourns-inc/CR0603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 -> https://www.digikey.de/de/products/detail/vishay-dale/CRCW0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; MFG Bourns Inc. -> YAGEO; MFG# CR0603AJ/-000EAS -> RC0603FR-07280RL
Connections:
- net +3.3VA: now also U6.10 (IO5)
- net CLKOUT: now also U6.20 (IO15); no longer U6.26 (IO20)
- net GND: now also D4.1 (K)
- net USB_D+: now also R33.2; no longer U6.18 (IO13)
- net USB_D-: now also R32.2; no longer U6.17 (IO12)
- net ~{CHARGE}: now also U6.19 (IO14); no longer U6.24 (IO18)
- net ~{WKUP}: now also U6.5 (IO2); no longer U6.28 (IO22)
- net SD.DETECT: now reaches U6.9 (IO4)
- net at U6.12 (IO0): now also R27.1
- net at U6.13 (IO1): now also R10.1
- net at R27.2: now also D4.2 (A)
- net HEARTBEAT renamed SDIO.DATA3
- net SDIO.DATA3: no longer R10.1
- net USB_DETECT renamed SDIO.CLK
- net ~{ALERT} renamed SDIO.DATA1
- new net: R32.1, U6.17 (IO12)
- new net: R33.1, U6.18 (IO13)
- new net SDIO.CMD: U6.24 (IO18)
- new net SDIO.DATA0: U6.26 (IO20)
- new net SDIO.DATA2: U6.28 (IO22)
- no-connect marks 3 -> 0
Other:
- added sheet 24V Supply (24v_supply.kicad_sch)
- added sheet I2C Devices (i2c_devices.kicad_sch)
- added sheet Power (power.kicad_sch)
- added sheet USB (usb.kicad_sch)
- added sheet uSD-Card (usd_card.kicad_sch)
- note added: "LP"
- note removed: "100nF !"
- note removed: "3.3V Reference Voltage"
- note removed: "3.3V Supply"
- note removed: "ADC"
- note removed: "FRAM"
- note removed: "I2C Temp."
- note removed: "I2C: 0x48"
- note removed: "I2C: 0x49"
- note removed: "I2C: 0x51"
- note removed: "I2C: 0x52"
- note removed: "IO2 !"
- note removed: "IO4 !"
- note removed: "I_{out,max} = 450 mA"
- note removed: "RTC"
- note removed: "USB/Power In"
- note removed: "USP Switch"
- moved on the sheet: C8, C9, D2, H1, H2, H3, H4, R10, R12, R19, R6, R8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
